Commit message: [panda_eus] add realsense and endeffector link

File: jsk_panda_robot/panda_eus/models/dual_panda.urdf.xacro (robot description, xacro)
@@ -308,3 +308,51 @@
     </plugin>
   </gazebo>
+  <!-- realsense -->
+  <link name="$(arg arm_id_1)_camera_link" >
+    <!-- <geometry> -->
+    <!--   <mesh filename="../../jsk_panda_accessories/realsense/realsense_with_mount.stl"/> -->
+    <!-- </geometry> -->
+    <inertial>
+      <origin xyz="0.0 0.0 0.0" rpt="0 0 0" />
+      <mass value = "0.005" />
+      <inertia ixx="0.0000000001" ixy="0.0000000001" ixz="0.0000000001"
+    	       iyy="0.0000000001" iyz="0.0000000001" izz="0.0000000001" />
+    </inertial>
+  </link>
+  <joint name="$(arg arm_id_1)_camera_joint" type="fixed">
+    <parent link="$(arg arm_id_1)_link7"/>
+    <child link="$(arg arm_id_1)_camera_link"/>
+    <origin xyz="0.049497475 -0.02828421 0.12375" rpy="1.57079632 -1.57079632 0.78539816"/>
+  </joint>
+  <link name="$(arg arm_id_2)_camera_link" >
+    <!-- <geometry> -->
+    <!--   <mesh filename="../../jsk_panda_accessories/realsense/realsense_with_mount.stl"/> -->
+    <!-- </geometry> -->
+    <inertial>
+      <origin xyz="0.0 0.0 0.0" rpt="0 0 0" />
+      <mass value = "0.005" />
+      <inertia ixx="0.0000000001" ixy="0.0000000001" ixz="0.0000000001"
+    	       iyy="0.0000000001" iyz="0.0000000001" izz="0.0000000001" />
+    </inertial>
+  </link>
+  <joint name="$(arg arm_id_2)_camera_joint" type="fixed">
+    <parent link="$(arg arm_id_2)_link7"/>
+    <child link="$(arg arm_id_2)_camera_link"/>
+    <origin xyz="0.049497475 -0.02828421 0.12375" rpy="1.57079632 -1.57079632 0.78539816"/>
+  </joint>
+  <!-- eus end effector link -->
+  <link name="$(arg arm_id_1)_end_effector" >
+  </link>
+  <joint name="$(arg arm_id_1)_end_effector_joint" type="fixed">
+    <parent link="$(arg arm_id_1)_link7"/>
+    <child link="$(arg arm_id_1)_end_effector"/>
+    <origin xyz="0 0 0.2" rpy="0 0 0"/>
+  </joint>
+  <link name="$(arg arm_id_2)_end_effector" >
+  </link>
+  <joint name="$(arg arm_id_2)_end_effector_joint" type="fixed">
+    <parent link="$(arg arm_id_2)_link7"/>
+    <child link="$(arg arm_id_2)_end_effector"/>
+    <origin xyz="0 0 0.2" rpy="0 0 0"/>
+  </joint>
 </robot>

Commit message: [panda_eus] fix pose of end_effector link

File: jsk_panda_robot/panda_eus/models/dual_panda.urdf.xacro (robot description, xacro)
@@ -347,5 +347,5 @@
     <parent link="$(arg arm_id_1)_link7"/>
     <child link="$(arg arm_id_1)_end_effector"/>
-    <origin xyz="0 0 0.2" rpy="0 0 0"/>
+    <origin xyz="0 0 0.2" rpy="0 -1.570796327 -0.785398163"/>
   </joint>
   <link name="$(arg arm_id_2)_end_effector" >
@@ -354,5 +354,5 @@
     <parent link="$(arg arm_id_2)_link7"/>
     <child link="$(arg arm_id_2)_end_effector"/>
-    <origin xyz="0 0 0.2" rpy="0 0 0"/>
+    <origin xyz="0 0 0.2" rpy="0 -1.570796327 -0.785398163"/>
   </joint>
 </robot>

Commit message: Commit changes stashed and uncommitted

File: jsk_panda_robot/panda_eus/models/dual_panda.urdf.xacro (robot description, xacro)
@@ -35,5 +35,5 @@
     -->
     <visual>
-      <origin xyz="0.3 0 0.71" />
+      <origin xyz="0.55 0 0.71" />
       <geometry>
         <box size="0.6 1.2 0.02" />
@@ -61,4 +61,24 @@
     <origin xyz="-0.08 0.0 0.8" rpy="0.0 0.0 0.0" />
   </joint>
+  <link name="workbench">
+   <visual>
+     <geometry>
+       <box size="0.5 0.5 0.01"/>
+     </geometry>
+     <material name="Workbench">
+       <color rgba="0.15 0.15 0.15 1.0"/>
+     </material>
+   </visual>
+   <collision>
+     <geometry>
+       <box size="0.5 0.5 0.01"/>
+     </geometry>
+   </collision>
+  </link>
+  <joint name="base_to_workbench" type="fixed">
+    <parent link="dual_arm_base"/>
+    <child  link="workbench"/>
+    <origin rpy="0.0 0.0 0.0" xyz="0.465 -0.150 1.145"/>
+  </joint>
   <!--link name="table_plane">
     <visual>
@@ -80,5 +100,5 @@
   <link name="controller_plane0">
     <visual>
-      <origin xyz="0.3 0 0.01" />
+      <origin xyz="0.55 0 0.01" />
       <geometry>
         <box size="0.6 0.8 0.02" />
@@ -115,5 +135,5 @@
   <link name="controller0">
     <visual>
-      <origin xyz="0.3 0 0.134" />
+      <origin xyz="0.55 0 0.134" />
       <geometry>
         <box size="0.475 0.423 0.268" />
